File: kicad/axof4_base_board/power.sch (KiCad schematic (older format))
At the start: 15 parts, among them J2 PJ-102A, U3 L7805CV, U4 LM1117MPX-3_3_NOPB, U5 LM1117MPX-3_3_NOPB

Commit message: work on kicad project
Parts:
- removed C24: 10u, symbol axof4_base_board-rescue:CP1_Small-Device
- removed C25: 330n, symbol axof4_base_board-rescue:C_Small-Device
- removed C26: 100n, symbol axof4_base_board-rescue:C_Small-Device
- removed D1: 1N4001-G, digikey-footprints:DO-41, symbol dk_Diodes-Rectifiers-Single:1N4001-G
- removed U3: L7805CV, digikey-footprints:TO-220-3, symbol dk_PMIC-Voltage-Regulators-Linear:L7805CV
- added C24: 10p, Capacitor_SMD:C_1206_3216Metric_Pad1.42x1.75mm_HandSolder, symbol axof4_base_board-rescue:C_Small-Device
- added C25, C26: 100u, Capacitor_SMD:CP_Elec_4x5.4, symbol axof4_base_board-rescue:CP1_Small-Device
- added C33: 100u, Capacitor_SMD:C_1206_3216Metric_Pad1.42x1.75mm_HandSolder, symbol axof4_base_board-rescue:CP1_Small-Device
- added C34: 10u, Capacitor_SMD:CP_Elec_4x5.4, symbol axof4_base_board-rescue:CP1_Small-Device
- added C35, C36: 220u, Capacitor_SMD:CP_Elec_4x5.4, symbol axof4_base_board-rescue:CP1_Small-Device
- added C37, C38: 100n, Capacitor_SMD:C_1206_3216Metric_Pad1.42x1.75mm_HandSolder, symbol axof4_base_board-rescue:C_Small-Device
- added D1: 1N4001, Diode_THT:D_DO-41_SOD81_P10.16mm_Horizontal, symbol Diode:1N4001
- added J3: power_sw, symbol axof4_base_board-rescue:Conn_01x02-Connector_Generic
- added U3: LT1054, symbol Regulator_SwitchedCapacitor:LT1054
- added U6: L7805, symbol Regulator_Linear:L7805
- added U7: L7905, symbol Regulator_Linear:L7905
- C28, C29, C30: footprint (none) -> Capacitor_SMD:CP_Elec_4x5.4
- C31, C32: footprint (none) -> Capacitor_SMD:C_1206_3216Metric_Pad1.42x1.75mm_HandSolder
Connections:
- net labels added: +3.3V-power, -5V
- wire segments 55 -> 109
- no-connect marks 0 -> 3
Other:
- note removed: "DC 9-12V IN"
- moved on the sheet: C27, C28, C29, C30, C31, C32, R25, U4, U5

Commit message: cleanup, dedicated PCB WIP
Parts:
- C27: footprint (none) -> Capacitor_SMD:CP_Elec_4x5.4
- J2: symbol dk_Barrel-Power-Connectors:PJ-102A -> axof4_base_board-rescue:PJ-102A-dk_Barrel-Power-Connectors
- J3: footprint (none) -> Connector_PinHeader_2.54mm:PinHeader_1x02_P2.54mm_Vertical
- R25: footprint (none) -> Resistor_SMD:R_1206_3216Metric_Pad1.42x1.75mm_HandSolder
- U3: footprint (none) -> Package_DIP:DIP-8_W7.62mm
- U4, U5: symbol dk_PMIC-Voltage-Regulators-Linear:LM1117MPX-3_3_NOPB -> axof4_base_board-rescue:LM1117MPX-3_3_NOPB-dk_PMIC-Voltage-Regulators-Linear
- U6, U7: footprint (none) -> Package_TO_SOT_THT:TO-220-3_Vertical
Changed lines of the file:
@@
 $Descr A4 11693 8268
 encoding utf-8
-Sheet 5 6
+Sheet 5 7
 Title ""
 Date ""
@@
 $EndComp
 $Comp
-L dk_PMIC-Voltage-Regulators-Linear:LM1117MPX-3_3_NOPB U4
+L axof4_base_board-rescue:LM1117MPX-3_3_NOPB-dk_PMIC-Voltage-Regulators-Linear U4
 U 1 1 5ED8D948
 P 8650 2650
@@
 $EndComp
 $Comp
-L dk_PMIC-Voltage-Regulators-Linear:LM1117MPX-3_3_NOPB U5
+L axof4_base_board-rescue:LM1117MPX-3_3_NOPB-dk_PMIC-Voltage-Regulators-Linear U5
 U 1 1 5ED8E22F
 P 8650 4000
@@
 F 0 "C27" H 7291 2846 50  0000 L CNN
 F 1 "1u" H 7291 2755 50  0000 L CNN
-F 2 "" H 7200 2800 50  0001 C CNN
+F 2 "Capacitor_SMD:CP_Elec_4x5.4" H 7200 2800 50  0001 C CNN
 F 3 "" H 7200 2800 50  0001 C CNN
 	1    7200 2800
@@
 F 0 "R25" V 7550 2650 50  0000 C CNN
 F 1 "4.7" V 7650 2650 50  0000 C CNN
-F 2 "" V 7580 2650 50  0001 C CNN
+F 2 "Resistor_SMD:R_1206_3216Metric_Pad1.42x1.75mm_HandSolder" V 7580 2650 50  0001 C CNN
 F 3 "" H 7650 2650 50  0001 C CNN
 	1    7650 2650
@@
 $EndComp
 $Comp
-L dk_Barrel-Power-Connectors:PJ-102A J2
+L axof4_base_board-rescue:PJ-102A-dk_Barrel-Power-Connectors J2
 U 1 1 5EE0EA4E
 P 1550 3250
+AR Path="/5EE0EA4E" Ref="J2"  Part="1"
+AR Path="/5ED86ED4/5EE0EA4E" Ref="J2"  Part="1"
 F 0 "J2" H 1483 3475 50  0000 C CNN
 F 1 "PJ-102A" H 1483 3384 50  0000 C CNN
@@
 F 0 "J3" V 1814 2762 50  0000 R CNN
 F 1 "power_sw" V 2000 3050 50  0000 R CNN
-F 2 "" H 1850 2950 50  0001 C CNN
+F 2 "Connector_PinHeader_2.54mm:PinHeader_1x02_P2.54mm_Vertical" H 1850 2950 50  0001 C CNN
 F 3 "" H 1850 2950 50  0001 C CNN
 	1    1850 2950
@@
 F 0 "U3" H 3200 4350 50  0000 C CNN
 F 1 "LT1054" H 3350 3400 50  0000 C CNN
-F 2 "" H 3250 3800 50  0001 C CNN
+F 2 "Package_DIP:DIP-8_W7.62mm" H 3250 3800 50  0001 C CNN
 F 3 "https://www.analog.com/media/en/technical-documentation/data-sheets/1054lfh.pdf" H 3250 3800 50  0001 C CNN
 	1    3150 3900
@@
 F 0 "U7" H 4550 3751 50  0000 C CNN
 F 1 "L7905" H 4550 3660 50  0000 C CNN
-F 2 "" H 4550 3700 50  0001 C CIN
+F 2 "Package_TO_SOT_THT:TO-220-3_Vertical" H 4550 3700 50  0001 C CIN
 F 3 "http://www.st.com/content/ccc/resource/technical/document/datasheet/c9/16/86/41/c7/2b/45/f2/CD00000450.pdf/files/CD00000450.pdf/jcr:content/translations/en.CD00000450.pdf" H 4550 3900 50  0001 C CNN
 	1    4550 3900
@@
 F 0 "U6" H 4550 3242 50  0000 C CNN
 F 1 "L7805" H 4550 3151 50  0000 C CNN
-F 2 "" H 4575 2850 50  0001 L CIN
+F 2 "Package_TO_SOT_THT:TO-220-3_Vertical" H 4575 2850 50  0001 L CIN
 F 3 "http://www.st.com/content/ccc/resource/technical/document/datasheet/41/4f/b3/b0/12/d4/47/88/CD00000444.pdf/files/CD00000444.pdf/jcr:content/translations/en.CD00000444.pdf" H 4550 2950 50  0001 C CNN
 	1    4550 3000
@@
 	1950 3600 2600 3600
 Wire Wire Line
-	2650 3250 3300 3250
+	2650 3250 2900 3250
 NoConn ~ 2750 3700
 Wire Wire Line
@@
 	3600 3800 3700 3800
 $Comp
-L power:PWR_FLAG #FLG0101
-U 1 1 5EF4839F
-P 800 1000
-F 0 "#FLG0101" H 800 1075 50  0001 C CNN
-F 1 "PWR_FLAG" H 800 1173 50  0000 C CNN
-F 2 "" H 800 1000 50  0001 C CNN
-F 3 "~" H 800 1000 50  0001 C CNN
-	1    800  1000
-	-1   0    0    1
-$EndComp
-$Comp
-L axof4_base_board-rescue:+5V-power #PWR0103
-U 1 1 5EF4B58B
-P 800 900
-F 0 "#PWR0103" H 800 750 50  0001 C CNN
-F 1 "+5V-power" H 815 1073 50  0000 C CNN
-F 2 "" H 800 900 50  0001 C CNN
-F 3 "" H 800 900 50  0001 C CNN
-	1    800  900
-	1    0    0    -1
-$EndComp
-Wire Wire Line
-	800  1000 800  900
-$Comp
-L power:-5V #PWR0104
-U 1 1 5EF5955F
-P 1250 900
-F 0 "#PWR0104" H 1250 1000 50  0001 C CNN
-F 1 "-5V" H 1265 1073 50  0000 C CNN
-F 2 "" H 1250 900 50  0001 C CNN
-F 3 "" H 1250 900 50  0001 C CNN
-	1    1250 900
-	1    0    0    -1
-$EndComp
-$Comp
-L axof4_base_board-rescue:+3.3V-power #PWR0105
-U 1 1 5EF5984D
-P 1750 900
-F 0 "#PWR0105" H 1750 750 50  0001 C CNN
-F 1 "+3.3V-power" H 1765 1073 50  0000 C CNN
-F 2 "" H 1750 900 50  0001 C CNN
-F 3 "" H 1750 900 50  0001 C CNN
-	1    1750 900
-	1    0    0    -1
-$EndComp
-$Comp
-L axof4_base_board-rescue:+3.3VA-power #PWR0106
-U 1 1 5EF59C31
-P 2400 900
-F 0 "#PWR0106" H 2400 750 50  0001 C CNN
-F 1 "+3.3VA-power" H 2415 1073 50  0000 C CNN
-F 2 "" H 2400 900 50  0001 C CNN
-F 3 "" H 2400 900 50  0001 C CNN
-	1    2400 900
-	1    0    0    -1
-$EndComp
-$Comp
-L power:PWR_FLAG #FLG0102
-U 1 1 5EF59FD9
-P 1250 1000
-F 0 "#FLG0102" H 1250 1075 50  0001 C CNN
-F 1 "PWR_FLAG" H 1250 1173 50  0000 C CNN
-F 2 "" H 1250 1000 50  0001 C CNN
-F 3 "~" H 1250 1000 50  0001 C CNN
-	1    1250 1000
-	-1   0    0    1
-$EndComp
-$Comp
-L power:PWR_FLAG #FLG0103
-U 1 1 5EF5A18D
-P 1750 1000
-F 0 "#FLG0103" H 1750 1075 50  0001 C CNN
-F 1 "PWR_FLAG" H 1750 1173 50  0000 C CNN
-F 2 "" H 1750 1000 50  0001 C CNN
-F 3 "~" H 1750 1000 50  0001 C CNN
-	1    1750 1000
-	-1   0    0    1
-$EndComp
-$Comp
-L power:PWR_FLAG #FLG0104
-U 1 1 5EF5A427
-P 2400 1000
-F 0 "#FLG0104" H 2400 1075 50  0001 C CNN
-F 1 "PWR_FLAG" H 2400 1173 50  0000 C CNN
-F 2 "" H 2400 1000 50  0001 C CNN
-F 3 "~" H 2400 1000 50  0001 C CNN
-	1    2400 1000
-	-1   0    0    1
-$EndComp
-Wire Wire Line
-	2400 1000 2400 900
-Wire Wire Line
-	1750 900  1750 1000
-Wire Wire Line
-	1250 900  1250 1000
-$Comp
-L axof4_base_board-rescue:GND-power #PWR?
-U 1 1 5EE201A1
-P 3000 850
-AR Path="/5ECDA234/5EE201A1" Ref="#PWR?"  Part="1"
-AR Path="/5ED86ED4/5EE201A1" Ref="#PWR0107"  Part="1"
-F 0 "#PWR0107" H 3000 600 50  0001 C CNN
-F 1 "GND" H 3005 677 50  0000 C CNN
-F 2 "" H 3000 850 50  0001 C CNN
-F 3 "" H 3000 850 50  0001 C CNN
-	1    3000 850
-	-1   0    0    1
-$EndComp
-$Comp
 L power:PWR_FLAG #FLG0105
 U 1 1 5EE20DCA
-P 3000 1000
-F 0 "#FLG0105" H 3000 1075 50  0001 C CNN
-F 1 "PWR_FLAG" H 3000 1173 50  0000 C CNN
-F 2 "" H 3000 1000 50  0001 C CNN
-F 3 "~" H 3000 1000 50  0001 C CNN
-	1    3000 1000
+P 1950 3700
+F 0 "#FLG0105" H 1950 3775 50  0001 C CNN
+F 1 "PWR_FLAG" H 1950 3873 50  0000 C CNN
+F 2 "" H 1950 3700 50  0001 C CNN
+F 3 "~" H 1950 3700 50  0001 C CNN
+	1    1950 3700
 	-1   0    0    1
 $EndComp
-Wire Wire Line
-	3000 850  3000 1000
+$Comp
+L power:PWR_FLAG #FLG0101
+U 1 1 5EEECED4
+P 2900 3050
+F 0 "#FLG0101" H 2900 3125 50  0001 C CNN
+F 1 "PWR_FLAG" H 2900 3223 50  0000 C CNN
+F 2 "" H 2900 3050 50  0001 C CNN
+F 3 "~" H 2900 3050 50  0001 C CNN
+	1    2900 3050
+	1    0    0    -1
+$EndComp
+Wire Wire Line
+	2900 3050 2900 3250
+Connection ~ 2900 3250
+Wire Wire Line
+	2900 3250 3300 3250
+Connection ~ 1950 3600
+Wire Wire Line
+	1950 3600 1950 3700
 $EndSCHEMATC

Commit message: rollback kicad project to use STM32F4DISCOVERY
Parts:
- C24, C31, C32, C33, C37, C38: footprint Capacitor_SMD:C_1206_3216Metric_Pad1.42x1.75mm_HandSolder -> Capacitor_SMD:C_0603_1608Metric
- C25, C26, C28, C29, C30, C34: footprint Capacitor_SMD:CP_Elec_4x5.4 -> Capacitor_SMD:CP_Elec_6.3x5.3
- D1: footprint Diode_THT:D_DO-41_SOD81_P10.16mm_Horizontal -> Diode_SMD:D_SOD-123
- R25: footprint Resistor_SMD:R_1206_3216Metric_Pad1.42x1.75mm_HandSolder -> Resistor_SMD:R_0603_1608Metric
Changed lines of the file:
@@
 F 0 "R25" V 7550 2650 50  0000 C CNN
 F 1 "4.7" V 7650 2650 50  0000 C CNN
-F 2 "Resistor_SMD:R_1206_3216Metric_Pad1.42x1.75mm_HandSolder" V 7580 2650 50  0001 C CNN
+F 2 "Resistor_SMD:R_0603_1608Metric" V 7580 2650 50  0001 C CNN
 F 3 "" H 7650 2650 50  0001 C CNN
 	1    7650 2650
@@
 F 0 "C28" H 8041 2846 50  0000 L CNN
 F 1 "10u" H 8041 2755 50  0000 L CNN
-F 2 "Capacitor_SMD:CP_Elec_4x5.4" H 7950 2800 50  0001 C CNN
+F 2 "Capacitor_SMD:CP_Elec_6.3x5.3" H 7950 2800 50  0001 C CNN
 F 3 "" H 7950 2800 50  0001 C CNN
 	1    7950 2800
@@
 F 0 "C31" H 9542 2796 50  0000 L CNN
 F 1 "100n" H 9542 2705 50  0000 L CNN
-F 2 "Capacitor_SMD:C_1206_3216Metric_Pad1.42x1.75mm_HandSolder" H 9450 2750 50  0001 C CNN
+F 2 "Capacitor_SMD:C_0603_1608Metric" H 9450 2750 50  0001 C CNN
 F 3 "" H 9450 2750 50  0001 C CNN
 	1    9450 2750
@@
 F 0 "C30" H 9241 4146 50  0000 L CNN
 F 1 "10u" H 9241 4055 50  0000 L CNN
-F 2 "Capacitor_SMD:CP_Elec_4x5.4" H 9150 4100 50  0001 C CNN
+F 2 "Capacitor_SMD:CP_Elec_6.3x5.3" H 9150 4100 50  0001 C CNN
 F 3 "" H 9150 4100 50  0001 C CNN
 	1    9150 4100
@@
 F 0 "C32" H 9542 4146 50  0000 L CNN
 F 1 "100n" H 9542 4055 50  0000 L CNN
-F 2 "Capacitor_SMD:C_1206_3216Metric_Pad1.42x1.75mm_HandSolder" H 9450 4100 50  0001 C CNN
+F 2 "Capacitor_SMD:C_0603_1608Metric" H 9450 4100 50  0001 C CNN
 F 3 "" H 9450 4100 50  0001 C CNN
 	1    9450 4100
@@
 F 0 "C29" H 9241 2796 50  0000 L CNN
 F 1 "10u" H 9241 2705 50  0000 L CNN
-F 2 "Capacitor_SMD:CP_Elec_4x5.4" H 9150 2750 50  0001 C CNN
+F 2 "Capacitor_SMD:CP_Elec_6.3x5.3" H 9150 2750 50  0001 C CNN
 F 3 "" H 9150 2750 50  0001 C CNN
 	1    9150 2750
@@
 F 0 "C34" H 4341 4496 50  0000 L CNN
 F 1 "10u" H 4341 4405 50  0000 L CNN
-F 2 "Capacitor_SMD:CP_Elec_4x5.4" H 4250 4450 50  0001 C CNN
+F 2 "Capacitor_SMD:CP_Elec_6.3x5.3" H 4250 4450 50  0001 C CNN
 F 3 "" H 4250 4450 50  0001 C CNN
 	1    4250 4450
@@
 F 0 "C25" H 3991 4496 50  0000 L CNN
 F 1 "100u" H 3991 4405 50  0000 L CNN
-F 2 "Capacitor_SMD:CP_Elec_4x5.4" H 3900 4450 50  0001 C CNN
+F 2 "Capacitor_SMD:CP_Elec_6.3x5.3" H 3900 4450 50  0001 C CNN
 F 3 "" H 3900 4450 50  0001 C CNN
 	1    3900 4450
@@
 F 0 "D1" H 2500 3033 50  0000 C CNN
 F 1 "1N4001" H 2500 3124 50  0000 C CNN
-F 2 "Diode_THT:D_DO-41_SOD81_P10.16mm_Horizontal" H 2500 3075 50  0001 C CNN
+F 2 "Diode_SMD:D_SOD-123" H 2500 3075 50  0001 C CNN
 F 3 "http://www.vishay.com/docs/88503/1n4001.pdf" H 2500 3250 50  0001 C CNN
 	1    2500 3250
@@
 F 0 "C37" H 5542 3246 50  0000 L CNN
 F 1 "100n" H 5542 3155 50  0000 L CNN
-F 2 "Capacitor_SMD:C_1206_3216Metric_Pad1.42x1.75mm_HandSolder" H 5450 3200 50  0001 C CNN
+F 2 "Capacitor_SMD:C_0603_1608Metric" H 5450 3200 50  0001 C CNN
 F 3 "" H 5450 3200 50  0001 C CNN
 	1    5450 3200
@@
 F 0 "C38" H 5542 3696 50  0000 L CNN
 F 1 "100n" H 5542 3605 50  0000 L CNN
-F 2 "Capacitor_SMD:C_1206_3216Metric_Pad1.42x1.75mm_HandSolder" H 5450 3650 50  0001 C CNN
+F 2 "Capacitor_SMD:C_0603_1608Metric" H 5450 3650 50  0001 C CNN
 F 3 "" H 5450 3650 50  0001 C CNN
 	1    5450 3650
@@
 F 0 "C26" H 4191 3246 50  0000 L CNN
 F 1 "100u" H 4191 3155 50  0000 L CNN
-F 2 "Capacitor_SMD:CP_Elec_4x5.4" H 4100 3200 50  0001 C CNN
+F 2 "Capacitor_SMD:CP_Elec_6.3x5.3" H 4100 3200 50  0001 C CNN
 F 3 "" H 4100 3200 50  0001 C CNN
 	1    4100 3200
@@
 F 0 "C33" H 4191 3696 50  0000 L CNN
 F 1 "100u" H 4191 3605 50  0000 L CNN
-F 2 "Capacitor_SMD:C_1206_3216Metric_Pad1.42x1.75mm_HandSolder" H 4100 3650 50  0001 C CNN
+F 2 "Capacitor_SMD:C_0603_1608Metric" H 4100 3650 50  0001 C CNN
 F 3 "" H 4100 3650 50  0001 C CNN
 	1    4100 3650
@@
 F 0 "C24" V 3250 4500 50  0000 L CNN
 F 1 "10p" V 3250 4700 50  0000 L CNN
-F 2 "Capacitor_SMD:C_1206_3216Metric_Pad1.42x1.75mm_HandSolder" H 3150 4650 50  0001 C CNN
+F 2 "Capacitor_SMD:C_0603_1608Metric" H 3150 4650 50  0001 C CNN
 F 3 "" H 3150 4650 50  0001 C CNN
 	1    3150 4650
