File: kicad/axof4_base_board/usb.sch (KiCad schematic (older format))
At the start: 2 parts

Commit message: kicad pcb backup, hohum axoctrl study
Parts:
- J12: renamed from J?; symbol Connector:USB_B -> axof4_base_board-rescue:USB_B-Connector
- gave numbers to parts that had none: 1
Changed lines of the file:
@@
 $EndDescr
 $Comp
-L Connector:USB_B J?
+L axof4_base_board-rescue:USB_B-Connector J?
 U 1 1 5F73AAFD
 P 5550 3750
-F 0 "J?" H 5607 4217 50  0000 C CNN
+AR Path="/5F73AAFD" Ref="J?"  Part="1"
+AR Path="/5F736ED6/5F73AAFD" Ref="J12"  Part="1"
+F 0 "J12" H 5607 4217 50  0000 C CNN
 F 1 "USB_B" H 5607 4126 50  0000 C CNN
 F 2 "" H 5700 3700 50  0001 C CNN
@@
 $EndComp
 $Comp
-L Power_Protection:USBLC6-2P6 U?
+L Power_Protection:USBLC6-2P6 U9
 U 1 1 5F73BA4A
 P 6550 3850
-F 0 "U?" V 6504 4294 50  0000 L CNN
+F 0 "U9" V 6504 4294 50  0000 L CNN
 F 1 "USBLC6-2P6" V 6595 4294 50  0000 L CNN
 F 2 "Package_TO_SOT_SMD:SOT-666" H 6550 3350 50  0001 C CNN

Commit message: rollback kicad project to use STM32F4DISCOVERY
Parts:
- J12: footprint (none) -> eec:GLOBAL_CONNECTOR_TECHNOLOGY-USB3145-30-1-A-0
Changed lines of the file:
@@
 F 0 "J12" H 5607 4217 50  0000 C CNN
 F 1 "USB_B" H 5607 4126 50  0000 C CNN
-F 2 "" H 5700 3700 50  0001 C CNN
+F 2 "eec:GLOBAL_CONNECTOR_TECHNOLOGY-USB3145-30-1-A-0" H 5700 3700 50  0001 C CNN
 F 3 " ~" H 5700 3700 50  0001 C CNN
 	1    5550 3750
