File: kicad/axof4_base_board_v0.2/codec.kicad_sch (KiCad schematic)
At the start: 23 parts, among them U1 CODECODER-WM8731SEDS_V(SSOP28), Y1 12.288MHz

Commit message: working towards own F427 daughterboard
Parts:
- R5: value 220 -> 33
Other:
- note added: "Fixed in v0.2: R6-R7 changed to 220 R8-R9 changed to 2.2k"
- note removed: "Fixed in v0.2: R5-R7 changed to 220 R8-R9 changed to 2.2k"
Changed lines of the file:
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@@
     (stroke (width 0) (type default) (color 0 0 0 0))
   )
-  (text "Fixed in v0.2:\nR5-R7 changed to 220\nR8-R9 changed to 2.2k"
+  (text "Fixed in v0.2:\nR6-R7 changed to 220\nR8-R9 changed to 2.2k"
     (at 195.58 100.33 0)
     (effects (font (size 2 2)) (justify left bottom))
@@
     (in_bom yes) (on_board yes)
     (property "Reference" "R5" (id 0) (at 181.61 76.835 90))
-    (property "Value" "220" (id 1) (at 181.61 78.74 90))
+    (property "Value" "33" (id 1) (at 181.61 78.74 90))
     (property "Footprint" "Resistor_SMD:R_0603_1608Metric_Pad0.98x0.95mm_HandSolder" (id 2) (at 181.61 76.962 90)
       (effects (font (size 1.27 1.27)) hide)
