File: kicad/axof4_base_board_v0.2/sdio.kicad_sch (KiCad schematic)
At the start: 7 parts, among them J1 Micro_SD_Card

Commit message: working towards own F427 daughterboard
Parts:
- J1: footprint foots:PJS008U-3000-0 -> foots:Sofng_TF-15x15_sd_card_socket
Other:
- note added: "v0.2: changed SD card socket to internal"
Changed lines of the file:
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@@
     (stroke (width 0) (type default) (color 0 0 0 0))
+  )
+  (text "v0.2:\nchanged SD card socket to internal" (at 166.37 76.2 0)
+    (effects (font (size 2 2)) (justify left bottom))
   )
   (global_label "SDIO_CK" (shape input) (at 98.425 106.68 180) (fields_autoplaced)
@@
     (property "Reference" "J1" (id 0) (at 182.88 85.9282 0))
     (property "Value" "Micro_SD_Card" (id 1) (at 182.88 88.2396 0))
-    (property "Footprint" "foots:PJS008U-3000-0" (id 2) (at 213.36 96.52 0)
-      (effects (font (size 1.27 1.27)) hide)
-    )
+    (property "Footprint" "foots:Sofng_TF-15x15_sd_card_socket" (id 2) (at 213.36 96.52 0)
+      (effects (font (size 1.27 1.27)) hide)
+    )
