File: kicad/axof4_base_board_v0.4/gate_io.kicad_sch (KiCad schematic)
At the start: 21 parts, among them J19 GATE_IN1, J20 GATE_IN2, J21 GATE_OUT1, J22 GATE_OUT2, Q1 MMBT3904, Q2 MMBT3904, U16 TL072

Commit message: revision 4
Parts:
- Q1, Q2: footprint Package_TO_SOT_SMD:SOT-23 -> Package_TO_SOT_SMD:SOT-23W
- R106, R107: value 51k -> 47k
- R108, R109: value 120k -> 100k
Other:
- note added: "0.0V to +3.3V"
- note added: "ca. +10.3V"
- note added: "turns active low at ca. +1.7V"
- note removed: "0.0V to +3.0V (or 3.3V? doesn't matter)"
- note removed: "ca. +10.0V"
- note removed: "turns on at ca. +2.0V"
- moved on the sheet: C58, C59, J19, J20, J21, J22, Q1, Q2, R100, R101, R102, R103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
