File: kicad/axof4_base_board_v0.4/power.kicad_sch (KiCad schematic)
At the start: 26 parts, among them J4 EURORACK_POWER, U10 LM317_TO-252, U3 LM4040DBZ-10, U4 LM317_TO-252

Commit message: revision 4
Parts:
- removed C11: 100nF, Capacitor_SMD:C_0603_1608Metric, symbol Device:C_Small
- removed FB3: 100 ohm @ 100 Mhz, Resistor_SMD:R_0805_2012Metric, symbol Device:FerriteBead_Small
- removed R19: 680, Resistor_SMD:R_0603_1608Metric, symbol Device:R
- removed U3: LM4040DBZ-10, Package_TO_SOT_SMD:SOT-23, symbol Reference_Voltage:LM4040DBZ-10
- added C67: 100nF, Capacitor_SMD:C_0603_1608Metric, symbol Device:C_Small
- added R58: 10k, Resistor_SMD:R_0603_1608Metric, symbol Device:R
- added R59: 3.3k, Resistor_SMD:R_0603_1608Metric, symbol Device:R
- added R72: 680, Resistor_SMD:R_0603_1608Metric, symbol Device:R
- added U18: CJ431, Package_TO_SOT_SMD:SOT-23W, symbol Reference_Voltage:TL432DBZ
- R56: value ? -> 240
- R57: value ? -> 750
Connections:
- net -12V: now also R72.1
- net AREF_-10V: now also C67.1, R59.1, R72.2, U18.3 (A)
- net GND: now also C67.2, R58.2, U18.2 (K)
- new net: R58.1, R59.2, U18.1 (REF)
Other:
- note added: "ca. 3.281V"
- note added: "ca. 5.156V"
- note added: "v0.4: added LM317 for 5V (mostly for usb host) replaced lm4040 with cj431 (basic part)"
- note removed: "fixed in v0.3: changed R16 to 680"
- note removed: "v0.5: added LM317 for 5V (basically only for usb host)"
