File: kicad/axof4_base_board_v0.4/usb.kicad_sch (KiCad schematic)
At the start: 17 parts, among them J23 Molex-105133, J24 GCT USB1040, U17 USBLC6-2P6, U5 AP2141, U8 USBLC6-2P6

Commit message: revision 4
Parts:
- R116: value 24k -> 47k
Connections:
- net +3V3 is gone; now on net +5V: R116.1
- net USB_HS_CONN_D+: now also U8.3 (I/O2); no longer U8.1 (I/O1)
- net USB_HS_CONN_D-: now also U8.1 (I/O1); no longer U8.3 (I/O2)
- net FS+: now reaches R54.2
- net FS+: now also U8.4 (I/O2); no longer U8.6 (I/O1)
- net FS-: now reaches R55.2
- net FS-: now also U8.6 (I/O1); no longer U8.4 (I/O2)
Other:
- note added: "5v voltage supervisor to PF10"
- note removed: "5v voltage supervisor to PF10 (fake 5V detection)"
- moved on the sheet: C61, C62
Changed lines of the file:
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@@
     (stroke (width 0) (type default) (color 0 0 0 0))
   )
-  (wire (pts (xy 194.31 107.95) (xy 190.5 107.95))
+  (wire (pts (xy 195.58 107.95) (xy 190.5 107.95))
     (stroke (width 0) (type default) (color 0 0 0 0))
   )
@@
     (stroke (width 0) (type default) (color 0 0 0 0))
   )
-  (wire (pts (xy 194.31 100.33) (xy 194.31 101.6))
+  (wire (pts (xy 195.58 100.33) (xy 195.58 101.6))
     (stroke (width 0) (type default) (color 0 0 0 0))
   )
@@
     (stroke (width 0) (type default) (color 0 0 0 0))
   )
-  (wire (pts (xy 194.31 100.33) (xy 186.69 100.33))
+  (wire (pts (xy 195.58 100.33) (xy 186.69 100.33))
     (stroke (width 0) (type default) (color 0 0 0 0))
   )
@@
     (stroke (width 0) (type default) (color 0 0 0 0))
   )
-  (wire (pts (xy 194.31 107.95) (xy 194.31 106.68))
+  (wire (pts (xy 195.58 107.95) (xy 195.58 106.68))
     (stroke (width 0) (type default) (color 0 0 0 0))
   )
@@
     (stroke (width 0) (type default) (color 0 0 0 0))
   )
-  (text "5v voltage supervisor to PF10\n(fake 5V detection)" (at 114.3 149.86 0)
+  (text "5v voltage supervisor to PF10" (at 114.3 149.86 0)
     (effects (font (size 1.27 1.27)) (justify left bottom))
   )
@@
     (effects (font (size 1.27 1.27)) (justify left bottom))
   )
+  (label "FS+" (at 228.6 99.06 0)
+    (effects (font (size 1.27 1.27)) (justify left bottom))
+  )
   (label "USB_HS_CONN_D+" (at 181.61 111.76 0)
     (effects (font (size 1.27 1.27)) (justify left bottom))
   )
   (label "USB_CONN_FS_D-" (at 45.72 97.79 0)
+    (effects (font (size 1.27 1.27)) (justify left bottom))
+  )
+  (label "FS-" (at 228.6 123.19 0)
     (effects (font (size 1.27 1.27)) (justify left bottom))
   )
@@
     (pin "6")
   )
-  (symbol (lib_id "Device:C_Small") (at 194.31 104.14 0) (unit 1)
-    (in_bom yes) (on_board yes)
-    (property "Reference" "C62" (id 0) (at 196.6468 102.9716 0)
-      (effects (font (size 1.27 1.27)) (justify left))
-    )
-    (property "Value" "100n" (id 1) (at 196.6468 105.283 0)
-      (effects (font (size 1.27 1.27)) (justify left))
-    )
-    (property "Footprint" "Capacitor_SMD:C_0603_1608Metric" (id 2) (at 194.31 104.14 0)
-      (effects (font (size 1.27 1.27)) hide)
-    )
-    (property "Datasheet" "~" (id 3) (at 194.31 104.14 0)
+  (symbol (lib_id "Device:C_Small") (at 186.69 104.14 0) (unit 1)
+    (in_bom yes) (on_board yes)
+    (property "Reference" "C62" (id 0) (at 189.0268 102.9716 0)
+      (effects (font (size 1.27 1.27)) (justify left))
+    )
+    (property "Value" "100n" (id 1) (at 189.0268 105.283 0)
+      (effects (font (size 1.27 1.27)) (justify left))
+    )
+    (property "Footprint" "Capacitor_SMD:C_0603_1608Metric" (id 2) (at 186.69 104.14 0)
+      (effects (font (size 1.27 1.27)) hide)
+    )
+    (property "Datasheet" "~" (id 3) (at 186.69 104.14 0)
       (effects (font (size 1.27 1.27)) hide)
     )
@@
     (pin "1")
   )
-  (symbol (lib_id "Device:C_Polarized_Small") (at 186.69 104.14 0) (unit 1)
-    (in_bom yes) (on_board yes)
-    (property "Reference" "C61" (id 0) (at 188.9252 102.9716 0)
-      (effects (font (size 1.27 1.27)) (justify left))
-    )
-    (property "Value" "47u" (id 1) (at 188.9252 105.283 0)
-      (effects (font (size 1.27 1.27)) (justify left))
-    )
-    (property "Footprint" "Capacitor_SMD:CP_Elec_6.3x5.4" (id 2) (at 186.69 104.14 0)
-      (effects (font (size 1.27 1.27)) hide)
-    )
-    (property "Datasheet" "~" (id 3) (at 186.69 104.14 0)
+  (symbol (lib_id "Device:C_Polarized_Small") (at 195.58 104.14 0) (unit 1)
+    (in_bom yes) (on_board yes)
+    (property "Reference" "C61" (id 0) (at 197.8152 102.9716 0)
+      (effects (font (size 1.27 1.27)) (justify left))
+    )
+    (property "Value" "47u" (id 1) (at 197.8152 105.283 0)
+      (effects (font (size 1.27 1.27)) (justify left))
+    )
+    (property "Footprint" "Capacitor_SMD:CP_Elec_6.3x5.4" (id 2) (at 195.58 104.14 0)
+      (effects (font (size 1.27 1.27)) hide)
+    )
+    (property "Datasheet" "~" (id 3) (at 195.58 104.14 0)
       (effects (font (size 1.27 1.27)) hide)
     )
@@
     (pin "5")
   )
-  (symbol (lib_id "power:+3.3V") (at 101.6 139.7 0) (unit 1)
-    (in_bom yes) (on_board yes) (fields_autoplaced)
-    (property "Reference" "#PWR0159" (id 0) (at 101.6 143.51 0)
-      (effects (font (size 1.27 1.27)) hide)
-    )
-    (property "Value" "+3.3V" (id 1) (at 101.6 136.1242 0))
-    (property "Footprint" "" (id 2) (at 101.6 139.7 0)
-      (effects (font (size 1.27 1.27)) hide)
-    )
-    (property "Datasheet" "" (id 3) (at 101.6 139.7 0)
-      (effects (font (size 1.27 1.27)) hide)
-    )
-    (pin "1")
-  )
   (symbol (lib_id "power:+5V") (at 186.69 76.2 0) (unit 1)
     (in_bom yes) (on_board yes)
@@
     (pin "1")
   )
+  (symbol (lib_id "power:+5V") (at 101.6 139.7 0) (unit 1)
+    (in_bom yes) (on_board yes)
+    (property "Reference" "#PWR0191" (id 0) (at 101.6 143.51 0)
+      (effects (font (size 1.27 1.27)) hide)
+    )
+    (property "Value" "+5V" (id 1) (at 101.981 135.3058 0))
+    (property "Footprint" "" (id 2) (at 101.6 139.7 0)
+      (effects (font (size 1.27 1.27)) hide)
+    )
+    (property "Datasheet" "" (id 3) (at 101.6 139.7 0)
+      (effects (font (size 1.27 1.27)) hide)
+    )
+    (pin "1")
+  )
   (symbol (lib_id "Device:R") (at 101.6 146.05 0) (unit 1)
     (in_bom yes) (on_board yes)
@@
       (effects (font (size 1.27 1.27)) (justify left))
     )
-    (property "Value" "24k" (id 1) (at 101.6 147.955 90)
+    (property "Value" "47k" (id 1) (at 101.6 147.955 90)
       (effects (font (size 1.27 1.27)) (justify left))
     )
@@
     (pin "2")
   )
-  (symbol (lib_id "Power_Protection:USBLC6-2P6") (at 226.06 111.76 270) (unit 1)
-    (in_bom yes) (on_board yes)
-    (property "Reference" "U8" (id 0) (at 234.95 107.95 90)
-      (effects (font (size 1.27 1.27)) (justify left))
-    )
-    (property "Value" "USBLC6-2P6" (id 1) (at 234.95 114.3 90)
+  (symbol (lib_id "Power_Protection:USBLC6-2P6") (at 226.06 111.76 270) (mirror x) (unit 1)
+    (in_bom yes) (on_board yes)
+    (property "Reference" "U8" (id 0) (at 234.95 115.57 90)
+      (effects (font (size 1.27 1.27)) (justify left))
+    )
+    (property "Value" "USBLC6-2P6" (id 1) (at 234.95 109.22 90)
       (effects (font (size 1.27 1.27)) (justify left))
     )
@@
       (effects (font (size 1.27 1.27)) hide)
     )
-    (property "Datasheet" "https://www.st.com/resource/en/datasheet/usblc6-2.pdf" (id 3) (at 234.95 116.84 0)
-      (effects (font (size 1.27 1.27)) hide)
-    )
+    (property "Datasheet" "https://www.st.com/resource/en/datasheet/usblc6-2.pdf" (id 3) (at 234.95 106.68 0)
+      (effects (font (size 1.27 1.27)) hide)
+    )
